File: Camera_Serializer/Power.kicad_sch (KiCad schematic)
At the start: 0 parts

Commit message: Finished POC circuit and added TVS diode
Parts:
- added C12: 100n, symbol Device:C
- added C18: 10n, symbol Device:C
- added D1: ~, symbol CameraServer_Symbols:PESD0402-240
- added J1: ~, symbol CameraServer_Symbols:7-2287906-0
- added L1: 560N, symbol Device:L
- added L2: 6u8, symbol Device:L
- added L3: 22u, symbol Device:L
- added R12, R13: 5k, symbol Device:R
- added TP4: TestPoint, symbol Connector:TestPoint
Connections:
- new net: L2.2, L3.1, R12.1, R13.2
- new net: L1.2, L2.1, R12.2
- new net +12V: C12.1, C18.1, L3.2, R13.1, TP4.1
- new net GND: C12.2, C18.2, D1.1, J1.2
- new net SIOP_COAX: D1.2, J1.1, L1.1

Commit message: Added CSI connector
Parts:
- D1: footprint (none) -> Diode_SMD:D_0402_1005Metric
Changed lines of the file:
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@@
 			)
 		)
-		(property "Footprint" ""
+		(property "Footprint" "Diode_SMD:D_0402_1005Metric"
 			(at 109.22 87.63 0)
 			(effects
@@
 			)
 		)
-		(property "Datasheet" ""
+		(property "Datasheet" "https://www.littelfuse.com/assetdocs/littelfuse-polymer-esd-suppressor-pesd-catalog-datasheet?assetguid=5186ff3a-844f-4b9e-926a-f506c7d3d551"
 			(at 109.22 87.63 0)
 			(effects
