File: Camera_Serializer/serializer.kicad_sch (KiCad schematic)
At the start: 32 parts

Commit message: Added 5V buck
Parts:
- TP1, TP2, TP3: footprint (none) -> TestPoint:TestPoint_Pad_D2.0mm
Changed lines of the file:
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@@
 			)
 		)
-		(property "Footprint" ""
+		(property "Footprint" "TestPoint:TestPoint_Pad_D2.0mm"
 			(at 231.14 88.9 0)
 			(effects
@@
 			)
 		)
-		(property "Footprint" ""
+		(property "Footprint" "TestPoint:TestPoint_Pad_D2.0mm"
 			(at 232.41 104.14 0)
 			(effects
@@
 			)
 		)
-		(property "Footprint" ""
+		(property "Footprint" "TestPoint:TestPoint_Pad_D2.0mm"
 			(at 232.41 101.6 0)
 			(effects

Commit message: Finishe schematic
Parts:
- C1, C10, C11, C13, C16, C17, C2, C3, C4, C5, C6, C7, C8, C9: footprint (none) -> Capacitor_SMD:C_0402_1005Metric_Pad0.74x0.62mm_HandSolder
- R10, R11, R2, R4, R6, R7, R8, R9: footprint (none) -> Resistor_SMD:R_0402_1005Metric_Pad0.72x0.64mm_HandSolder
- TP1, TP2, TP3: footprint TestPoint:TestPoint_Pad_D2.0mm -> TestPoint:TestPoint_Pad_D1.0mm
- U1: footprint Package_DFN_QFN:TQFN-32-1EP_5x5mm_P0.5mm_EP3.1x3.1mm -> CameraServer_Footprints:QFN50P500X500X80-33N; symbol analog_devices_gmsl:MAX96717GTJ -> CameraServer_Symbols:MAX96717GTJ_VY+; Arrow Part Number (none) -> MAX96717GTJ/VY+; Arrow Price/Stock (none) -> https://www.arrow.com/en/products/max96717gtjvy/analog-devi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; Height (none) -> 0.8; Manufacturer_Name (none) -> Analog Devices; Manufacturer_Part_Number (none) -> MAX96717GTJ/VY+; Mouser Part Number (none) -> 700-MAX96717GTJ/VY+; Mouser Price/Stock (none) -> https://www.mouser.co.uk/ProductDetail/Analog-Devices-Maxim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
- Y1: footprint (none) -> CameraServer_Footprints:EB2532YA08-25.000M_TR; symbol EB2532YA08-25.000M_TR:EB2532YA08-25.000M_TR -> CameraServer_Symbols:EB2532YA08-25.000M_TR; Height (none) -> 0.8; Manufacturer_Name (none) -> Ecliptek; Manufacturer_Part_Number (none) -> EB2532YA08-25.000M TR; Mouser Part Number (none) -> 669-EB2532YA08-25T; Mouser Price/Stock (none) -> https://www.mouser.co.uk/ProductDetail/Ecliptek-Abracon/EB2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
Connections:
- net GND: now also U1.33 (GND), Y1.4; no longer U1. (EP)
Other:
- moved on the sheet: C13, C17, TP1, TP2, TP3, U1
