File: Camera_Serializer/Camera_serializer.kicad_pcb (KiCad board)
At the start: 4 copper layers, 38.1 x 38.1 mm, 88 parts, among them J2 F32Q-1A7H1-11022, Q1 BSS138, Q2 BSS138, U2 PUSB3FR4Z, U3 TPS62133RGTR, U4 TPS62131RGTT, U5 TPS73601DBVR, U6 MIC5528-3.3YMT-TR

Commit message: Final hardware as of order
Parts:
- added T1: ~, CameraServer_Footprints:Coax Testpoint, F.Cu at (154.4, 89.5)
- J1: footprint CameraServer_Footprints:7-2287906-0 -> CameraServer_Footprints:RF55-28Z-T-00-50-G-SH
- turned J1 to 90 degrees
Routing:
- net /GMSL_Connector/SIOP_COAX: track 22.6 -> 17.1 mm
- net /csi/CSI.D2_N: track 24.6 -> 27.4 mm
- net /csi/CSI.D2_P: track 24.6 -> 27.4 mm
- net /csi/CSI.D3_P: track 24.6 -> 27.3 mm
- net /csi/CSI.D3_N: track 24.6 -> 27.2 mm
- net /csi/CSI.CK_P: track 27.7 -> 30.4 mm
- net /csi/CSI.D1_P: track 24.6 -> 27.3 mm
- net /csi/CSI.CK_N: track 27.7 -> 30.3 mm
- net GND: track 99.3 -> 96.7 mm, vias 66 -> 75
- net /csi/CSI.D0_P: track 24.6 -> 27.2 mm
- net /csi/CSI.D1_N: track 24.7 -> 26.7 mm
- net Net-(U1-MFP6): track 8.52 -> 9.07 mm
- net /csi/CSI.D0_N: track 24.6 -> 25.1 mm
Other:
- board text added: "Camera Serializer Rev2 Mars Rover Design Team Missouri S&T, 2026 Jesse Deuel"
- board text added: "Using Board stackup JLC04161H-3313"
- board text removed: "Camera Serializer Rev1 Mars Rover Design Team Missouri S&T, 2025 Jesse Deuel"
