File: Camera_Serializer/GMSL_Connector.kicad_sch (KiCad schematic)
At the start: 10 parts

Commit message: Finishe schematic
Parts:
- C12, C18: footprint (none) -> Capacitor_SMD:C_0402_1005Metric_Pad0.74x0.62mm_HandSolder
- J1: footprint (none) -> CameraServer_Footprints:7-2287906-0
- L1: value 560N -> 560n; footprint (none) -> CameraServer_Footprints:PFL1609-561MEW
- L2: footprint (none) -> CameraServer_Footprints:1812PS-682JRC
- L3: footprint (none) -> CameraServer_Footprints:SRN3015C-220M
- R12, R13: footprint (none) -> Resistor_SMD:R_0402_1005Metric_Pad0.72x0.64mm_HandSolder
- TP4: footprint TestPoint:TestPoint_Pad_D2.0mm -> TestPoint:TestPoint_Pad_D1.0mm
Connections:
- net GND: now also J1. (5)
Changed lines of the file:
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@@
+	)
+	(junction
+		(at 215.9 78.74)
+		(diameter 0)
+		(color 0 0 0 0)
 	)
 	(junction
@@
 	(wire
 		(pts
-			(xy 209.55 71.12) (xy 209.55 78.74)
+			(xy 222.25 71.12) (xy 222.25 78.74)
 		)
 		(stroke
@@
 	(wire
 		(pts
-			(xy 204.47 78.74) (xy 209.55 78.74)
+			(xy 204.47 78.74) (xy 215.9 78.74)
 		)
 		(stroke
@@
 		(pts
 			(xy 163.83 87.63) (xy 166.37 87.63)
+		)
+		(stroke
+			(width 0)
+			(type default)
+		)
+	)
+	(wire
+		(pts
+			(xy 215.9 78.74) (xy 222.25 78.74)
 		)
 		(stroke
@@
 			)
 		)
-		(property "Footprint" ""
+		(property "Footprint" "Resistor_SMD:R_0402_1005Metric_Pad0.72x0.64mm_HandSolder"
 			(at 160.02 85.852 90)
 			(effects
@@
 				(path "/ebaf1619-da94-4b8e-b57a-a386470e666e/602efbe5-ec9c-4bfc-a3ee-5e96e644a054"
 					(reference "R12")
+					(unit 1)
+				)
+			)
+		)
+	)
+	(symbol
+		(lib_id "power:PWR_FLAG")
+		(at 215.9 78.74 0)
+		(unit 1)
+		(exclude_from_sim no)
+		(in_bom yes)
+		(on_board yes)
+		(dnp no)
+		(fields_autoplaced yes)
+		(property "Reference" "#FLG01"
+			(at 215.9 76.835 0)
+			(effects
+				(font
+					(size 1.27 1.27)
+				)
+				(hide yes)
+			)
+		)
+		(property "Value" "PWR_FLAG"
+			(at 215.9 73.66 0)
+			(effects
+				(font
+					(size 1.27 1.27)
+				)
+			)
+		)
+		(property "Footprint" ""
+			(at 215.9 78.74 0)
+			(effects
+				(font
+					(size 1.27 1.27)
+				)
+				(hide yes)
+			)
+		)
+		(property "Datasheet" "~"
+			(at 215.9 78.74 0)
+			(effects
+				(font
+					(size 1.27 1.27)
+				)
+				(hide yes)
+			)
+		)
+		(property "Description" "Special symbol for telling ERC where power comes from"
+			(at 215.9 78.74 0)
+			(effects
+				(font
+					(size 1.27 1.27)
+				)
+				(hide yes)
+			)
+		)
+		(pin "1"
+		)
+		(instances
+			(project ""
+				(path "/ebaf1619-da94-4b8e-b57a-a386470e666e/602efbe5-ec9c-4bfc-a3ee-5e96e644a054"
+					(reference "#FLG01")
 					(unit 1)
 				)
@@
 	(symbol
 		(lib_id "power:+12V")
-		(at 209.55 71.12 0)
+		(at 222.25 71.12 0)
 		(unit 1)
 		(exclude_from_sim no)
@@
 		(fields_autoplaced yes)
 		(property "Reference" "#PWR020"
-			(at 209.55 74.93 0)
+			(at 222.25 74.93 0)
 			(effects
 				(font
@@
 		)
 		(property "Value" "+12V"
-			(at 209.55 66.04 0)
+			(at 222.25 66.04 0)
 			(effects
 				(font
@@
 		)
 		(property "Footprint" ""
-			(at 209.55 71.12 0)
+			(at 222.25 71.12 0)
 			(effects
 				(font
@@
 		)
 		(property "Datasheet" ""
-			(at 209.55 71.12 0)
+			(at 222.25 71.12 0)
 			(effects
 				(font
@@
 		)
 		(property "Description" "Power symbol creates a global label with name \"+12V\""
-			(at 209.55 71.12 0)
+			(at 222.25 71.12 0)
 			(effects
 				(font
@@
 			)
 		)
-		(property "Value" "560N"
+		(property "Value" "560n"
 			(at 147.32 76.2 90)
 			(effects
@@
 			)
 		)
-		(property "Footprint" ""
+		(property "Footprint" "CameraServer_Footprints:PFL1609-561MEW"
 			(at 147.32 78.74 0)
 			(effects
@@
 			)
 		)
-		(property "Datasheet" "~"
+		(property "Datasheet" "https://www.coilcraft.com/getmedia/2f4cd442-d64d-4413-a518-12fcfd03318d/pfl1609.pdf"
 			(at 147.32 78.74 0)
 			(effects
@@
 			)
 		)
-		(property "Footprint" "TestPoint:TestPoint_Pad_D2.0mm"
+		(property "Footprint" "TestPoint:TestPoint_Pad_D1.0mm"
 			(at 191.77 76.2 0)
 			(effects
@@
 			)
 		)
-		(property "Footprint" ""
+		(property "Footprint" "Capacitor_SMD:C_0402_1005Metric_Pad0.74x0.62mm_HandSolder"
 			(at 205.4352 87.63 0)
 			(effects
@@
 			)
 		)
-		(property "Footprint" ""
+		(property "Footprint" "CameraServer_Footprints:1812PS-682JRC"
 			(at 160.02 78.74 0)
 			(effects
@@
 			)
 		)
-		(property "Datasheet" "~"
+		(property "Datasheet" "https://www.coilcraft.com/getmedia/679e8dc0-2b0f-4b24-bc7a-b80ee286146a/1812ps.pdf"
 			(at 160.02 78.74 0)
 			(effects
@@
 			)
 		)
-		(property "Footprint" ""
+		(property "Footprint" "Capacitor_SMD:C_0402_1005Metric_Pad0.74x0.62mm_HandSolder"
 			(at 192.7352 87.63 0)
 			(effects
@@
 			)
 		)
-		(property "Footprint" ""
+		(property "Footprint" "CameraServer_Footprints:SRN3015C-220M"
 			(at 172.72 78.74 0)
 			(effects
@@
 		(on_board yes)
 		(dnp no)
-		(fields_autoplaced yes)
 		(property "Reference" "J1"
-			(at 95.25 72.39 0)
+			(at 95.25 74.422 0)
 			(effects
 				(font
@@
 			)
 		)
-		(property "Footprint" ""
+		(property "Footprint" "CameraServer_Footprints:7-2287906-0"
 			(at 95.25 78.74 0)
 			(effects
@@
 		)
 		(pin "2"
+		)
+		(pin ""
+		)
+		(pin ""
+		)
+		(pin ""
 		)
 		(instances
@@
 			)
 		)
-		(property "Footprint" ""
+		(property "Footprint" "Resistor_SMD:R_0402_1005Metric_Pad0.72x0.64mm_HandSolder"
 			(at 172.72 85.852 90)
 			(effects

Commit message: Finished routing
Connections:
- net GND: now also J1.3, J1.4, J1.5; no longer J1. (5)
Changed lines of the file:
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@@
 		(pin "2"
 		)
-		(pin ""
+		(pin "5"
 		)
-		(pin ""
+		(pin "4"
 		)
-		(pin ""
+		(pin "3"
 		)
 		(instances

Commit message: Updated to Kicad 9 and added datasheet for 22uH inductor
Changed lines of the file:
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@@
 (kicad_sch
-	(version 20231120)
+	(version 20250114)
 	(generator "eeschema")
-	(generator_version "8.0")
+	(generator_version "9.0")
 	(paper "A4")
 	(junction
@@
 			)
 		)
-		(property "Datasheet" "~"
+		(property "Datasheet" "https://www.bourns.com/docs/product-datasheets/SRN3015C.pdf"
 			(at 172.72 78.74 0)
 			(effects

Commit message: Final hardware as of order
Parts:
- added T1: ~, CameraServer_Footprints:Coax Testpoint, symbol CameraServer_Symbols:Coax_Test_Point
- J1: footprint CameraServer_Footprints:7-2287906-0 -> CameraServer_Footprints:RF55-28Z-T-00-50-G-SH; symbol CameraServer_Symbols:7-2287906-0 -> CameraServer_Symbols:RF55-28Z-T-00-50-G-SH
Connections:
- net GND: now also T1.2
- net SIOP_COAX: now also T1.1
Changed lines of the file:
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@@
+	)
+	(junction
+		(at 133.35 78.74)
+		(diameter 0)
+		(color 0 0 0 0)
 	)
 	(junction
@@
 	(wire
 		(pts
-			(xy 109.22 78.74) (xy 143.51 78.74)
+			(xy 109.22 78.74) (xy 133.35 78.74)
 		)
 		(stroke
@@
 	(wire
 		(pts
+			(xy 130.81 72.39) (xy 130.81 73.66)
+		)
+		(stroke
+			(width 0)
+			(type default)
+		)
+	)
+	(wire
+		(pts
 			(xy 186.69 76.2) (xy 186.69 78.74)
 		)
@@
 	(wire
 		(pts
+			(xy 133.35 69.85) (xy 133.35 78.74)
+		)
+		(stroke
+			(width 0)
+			(type default)
+		)
+	)
+	(wire
+		(pts
 			(xy 156.21 87.63) (xy 154.94 87.63)
 		)
@@
 		(pts
 			(xy 151.13 78.74) (xy 154.94 78.74)
+		)
+		(stroke
+			(width 0)
+			(type default)
+		)
+	)
+	(wire
+		(pts
+			(xy 133.35 78.74) (xy 143.51 78.74)
 		)
 		(stroke
@@
 		)
 		(instances
-			(project ""
+			(project "Camera_serializer"
 				(path "/ebaf1619-da94-4b8e-b57a-a386470e666e/602efbe5-ec9c-4bfc-a3ee-5e96e644a054"
 					(reference "#FLG01")
@@
 	)
 	(symbol
+		(lib_id "power:GND")
+		(at 130.81 73.66 0)
+		(unit 1)
+		(exclude_from_sim no)
+		(in_bom yes)
+		(on_board yes)
+		(dnp no)
+		(property "Reference" "#PWR059"
+			(at 130.81 80.01 0)
+			(effects
+				(font
+					(size 1.27 1.27)
+				)
+				(hide yes)
+			)
+		)
+		(property "Value" "GND"
+			(at 126.746 75.438 0)
+			(effects
+				(font
+					(size 1.27 1.27)
+				)
+			)
+		)
+		(property "Footprint" ""
+			(at 130.81 73.66 0)
+			(effects
+				(font
+					(size 1.27 1.27)
+				)
+				(hide yes)
+			)
+		)
+		(property "Datasheet" ""
+			(at 130.81 73.66 0)
+			(effects
+				(font
+					(size 1.27 1.27)
+				)
+				(hide yes)
+			)
+		)
+		(property "Description" "Power symbol creates a global label with name \"GND\" , ground"
+			(at 130.81 73.66 0)
+			(effects
+				(font
+					(size 1.27 1.27)
+				)
+				(hide yes)
+			)
+		)
+		(pin "1"
+		)
+		(instances
+			(project "Camera_serializer"
+				(path "/ebaf1619-da94-4b8e-b57a-a386470e666e/602efbe5-ec9c-4bfc-a3ee-5e96e644a054"
+					(reference "#PWR059")
+					(unit 1)
+				)
+			)
+		)
+	)
+	(symbol
 		(lib_id "Device:L")
 		(at 160.02 78.74 90)
@@
 	)
 	(symbol
-		(lib_id "CameraServer_Symbols:7-2287906-0")
+		(lib_id "CameraServer_Symbols:Coax_Test_Point")
+		(at 133.35 66.04 0)
+		(unit 1)
+		(exclude_from_sim no)
+		(in_bom yes)
+		(on_board yes)
+		(dnp no)
+		(fields_autoplaced yes)
+		(property "Reference" "T1"
+			(at 138.43 64.7699 0)
+			(effects
+				(font
+					(size 1.27 1.27)
+				)
+				(justify left)
+			)
+		)
+		(property "Value" "~"
+			(at 138.43 67.3099 0)
+			(effects
+				(font
+					(size 1.27 1.27)
+				)
+				(justify left)
+			)
+		)
+		(property "Footprint" "CameraServer_Footprints:Coax Testpoint"
+			(at 133.35 66.04 0)
+			(effects
+				(font
+					(size 1.27 1.27)
+				)
+				(hide yes)
+			)
+		)
+		(property "Datasheet" ""
+			(at 133.35 66.04 0)
+			(effects
+				(font
+					(size 1.27 1.27)
+				)
+				(hide yes)
+			)
+		)
+		(property "Description" ""
+			(at 133.35 66.04 0)
+			(effects
+				(font
+					(size 1.27 1.27)
+				)
+				(hide yes)
+			)
+		)
+		(pin "2"
+		)
+		(pin "1"
+		)
+		(instances
+			(project "Camera_serializer"
+				(path "/ebaf1619-da94-4b8e-b57a-a386470e666e/602efbe5-ec9c-4bfc-a3ee-5e96e644a054"
+					(reference "T1")
+					(unit 1)
+				)
+			)
+		)
+	)
+	(symbol
+		(lib_id "CameraServer_Symbols:RF55-28Z-T-00-50-G-SH")
 		(at 95.25 78.74 0)
 		(unit 1)
@@
 			)
 		)
-		(property "Footprint" "CameraServer_Footprints:7-2287906-0"
+		(property "Footprint" "CameraServer_Footprints:RF55-28Z-T-00-50-G-SH"
 			(at 95.25 78.74 0)
 			(effects
