File: Camera_Serializer/power_converters.kicad_sch (KiCad schematic)
At the start: 35 parts, among them Q1 BSS138, Q2 BSS138, U3 TPS62133RGTR, U4 TPS62131RGTT, U5 TPS73601DBVR, U6 MIC5528-3.3YMT-TR

Commit message: Final hardware as of order
Changed lines of the file:
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@@
 	)
 	(junction
+		(at 193.04 49.53)
+		(diameter 0)
+		(color 0 0 0 0)
+	)
+	(junction
 		(at 92.71 67.31)
 		(diameter 0)
@@
 	)
 	(junction
-		(at 193.04 49.53)
-		(diameter 0)
-		(color 0 0 0 0)
-	)
-	(junction
 		(at 92.71 152.4)
 		(diameter 0)
@@
 	(wire
 		(pts
+			(xy 193.04 46.99) (xy 193.04 49.53)
+		)
+		(stroke
+			(width 0)
+			(type default)
+		)
+	)
+	(wire
+		(pts
 			(xy 101.6 39.37) (xy 101.6 43.18)
 		)
@@
 	(wire
 		(pts
-			(xy 193.04 49.53) (xy 193.04 52.07)
-		)
-		(stroke
-			(width 0)
-			(type default)
-		)
-	)
-	(wire
-		(pts
 			(xy 269.24 40.64) (xy 269.24 43.18)
 		)
@@
 	(wire
 		(pts
+			(xy 193.04 49.53) (xy 193.04 52.07)
+		)
+		(stroke
+			(width 0)
+			(type default)
+		)
+	)
+	(wire
+		(pts
 			(xy 87.63 44.45) (xy 87.63 41.91)
 		)
@@
 	(wire
 		(pts
+			(xy 193.04 49.53) (xy 195.58 49.53)
+		)
+		(stroke
+			(width 0)
+			(type default)
+		)
+	)
+	(wire
+		(pts
 			(xy 86.36 154.94) (xy 92.71 154.94)
 		)
@@
 	(wire
 		(pts
+			(xy 195.58 52.07) (xy 193.04 52.07)
+		)
+		(stroke
+			(width 0)
+			(type default)
+		)
+	)
+	(wire
+		(pts
 			(xy 86.36 49.53) (xy 97.79 49.53)
 		)
@@
 	(wire
 		(pts
-			(xy 193.04 46.99) (xy 193.04 49.53)
-		)
-		(stroke
-			(width 0)
-			(type default)
-		)
-	)
-	(wire
-		(pts
 			(xy 144.78 124.46) (xy 144.78 127)
 		)
@@
 	(wire
 		(pts
-			(xy 193.04 49.53) (xy 195.58 49.53)
-		)
-		(stroke
-			(width 0)
-			(type default)
-		)
-	)
-	(wire
-		(pts
 			(xy 35.56 57.15) (xy 25.4 57.15)
 		)
@@
 	(wire
 		(pts
-			(xy 193.04 52.07) (xy 195.58 52.07)
-		)
-		(stroke
-			(width 0)
-			(type default)
-		)
-	)
-	(wire
-		(pts
 			(xy 101.6 39.37) (xy 107.95 39.37)
 		)
@@
 		)
 		(instances
-			(project ""
+			(project "Camera_serializer"
 				(path "/ebaf1619-da94-4b8e-b57a-a386470e666e/aa1b48ff-d467-42b0-a250-5333a1eca37c"
 					(reference "D2")
@@
 		)
 		(instances
-			(project ""
+			(project "Camera_serializer"
 				(path "/ebaf1619-da94-4b8e-b57a-a386470e666e/aa1b48ff-d467-42b0-a250-5333a1eca37c"
 					(reference "D3")
@@
 		)
 		(instances
-			(project ""
+			(project "Camera_serializer"
 				(path "/ebaf1619-da94-4b8e-b57a-a386470e666e/aa1b48ff-d467-42b0-a250-5333a1eca37c"
 					(reference "U4")
@@
 		)
 		(instances
-			(project ""
+			(project "Camera_serializer"
 				(path "/ebaf1619-da94-4b8e-b57a-a386470e666e/aa1b48ff-d467-42b0-a250-5333a1eca37c"
 					(reference "Q1")
@@
 		)
 		(instances
-			(project ""
+			(project "Camera_serializer"
 				(path "/ebaf1619-da94-4b8e-b57a-a386470e666e/aa1b48ff-d467-42b0-a250-5333a1eca37c"
 					(reference "C20")
@@
 		)
 		(instances
-			(project ""
+			(project "Camera_serializer"
 				(path "/ebaf1619-da94-4b8e-b57a-a386470e666e/aa1b48ff-d467-42b0-a250-5333a1eca37c"
 					(reference "L4")
@@
 		)
 		(instances
-			(project ""
+			(project "Camera_serializer"
 				(path "/ebaf1619-da94-4b8e-b57a-a386470e666e/aa1b48ff-d467-42b0-a250-5333a1eca37c"
 					(reference "U3")
@@
 		)
 		(instances
-			(project ""
+			(project "Camera_serializer"
 				(path "/ebaf1619-da94-4b8e-b57a-a386470e666e/aa1b48ff-d467-42b0-a250-5333a1eca37c"
 					(reference "#PWR032")
@@
 		)
 		(instances
-			(project ""
+			(project "Camera_serializer"
 				(path "/ebaf1619-da94-4b8e-b57a-a386470e666e/aa1b48ff-d467-42b0-a250-5333a1eca37c"
 					(reference "R20")
@@
 		)
 		(instances
-			(project ""
+			(project "Camera_serializer"
 				(path "/ebaf1619-da94-4b8e-b57a-a386470e666e/aa1b48ff-d467-42b0-a250-5333a1eca37c"
 					(reference "TP5")
@@
 		)
 		(instances
-			(project ""
+			(project "Camera_serializer"
 				(path "/ebaf1619-da94-4b8e-b57a-a386470e666e/aa1b48ff-d467-42b0-a250-5333a1eca37c"
 					(reference "U5")
@@
 		)
 		(instances
-			(project ""
+			(project "Camera_serializer"
 				(path "/ebaf1619-da94-4b8e-b57a-a386470e666e/aa1b48ff-d467-42b0-a250-5333a1eca37c"
 					(reference "C27")
@@
 		)
 		(instances
-			(project ""
+			(project "Camera_serializer"
 				(path "/ebaf1619-da94-4b8e-b57a-a386470e666e/aa1b48ff-d467-42b0-a250-5333a1eca37c"
 					(reference "R21")
@@
 		)
 		(instances
-			(project ""
+			(project "Camera_serializer"
 				(path "/ebaf1619-da94-4b8e-b57a-a386470e666e/aa1b48ff-d467-42b0-a250-5333a1eca37c"
 					(reference "U6")
@@
 		)
 		(instances
-			(project ""
+			(project "Camera_serializer"
 				(path "/ebaf1619-da94-4b8e-b57a-a386470e666e/aa1b48ff-d467-42b0-a250-5333a1eca37c"
 					(reference "#PWR042")
@@
 		)
 		(instances
-			(project ""
+			(project "Camera_serializer"
 				(path "/ebaf1619-da94-4b8e-b57a-a386470e666e/aa1b48ff-d467-42b0-a250-5333a1eca37c"
 					(reference "R18")
@@
 		)
 		(instances
-			(project ""
+			(project "Camera_serializer"
 				(path "/ebaf1619-da94-4b8e-b57a-a386470e666e/aa1b48ff-d467-42b0-a250-5333a1eca37c"
 					(reference "#PWR034")
